File: pcb/MagneticLevitator/MagneticLevitator.kicad_pcb (KiCad board)
At the start: 2 copper layers, 112.8 x 75.8 mm, 12 parts, among them J1 ESP32 Left Side Pins, J2 ESP32 Right Side Pins, J3 Screw_Terminal_01x02, J4 Screw_Terminal_01x02, J5 ACS712T Breakout, J6 hall effect sensor breakout, Q1 Q_NMOS_GDS

Commit message: more pcb updates
Parts:
- removed 1.8K: 1.8k, Resistor_THT:R_Axial_DIN0207_L6.3mm_D2.5mm_P10.16mm_Horizontal
- removed 10K: 10k, Resistor_THT:R_Axial_DIN0207_L6.3mm_D2.5mm_P10.16mm_Horizontal
- removed 220R: 220, Resistor_THT:R_Axial_DIN0207_L6.3mm_D2.5mm_P10.16mm_Horizontal
- removed 3.3K: 3.3k, Resistor_THT:R_Axial_DIN0207_L6.3mm_D2.5mm_P10.16mm_Horizontal
- removed D1: D, Diode_THT:D_DO-41_SOD81_P7.62mm_Horizontal
- removed J5: ACS712T Breakout, Connector_PinSocket_2.54mm:PinSocket_1x03_P2.54mm_Vertical
- added C1: 100uF, Capacitor_THT:CP_Radial_D6.3mm_P2.50mm, F.Cu at (111.5, 119.5)
- added C2: 10uF, Capacitor_THT:CP_Radial_D6.3mm_P2.50mm, F.Cu at (137.0, 120.5)
- added C3: 100nF, Capacitor_THT:C_Disc_D3.0mm_W1.6mm_P2.50mm, F.Cu at (148.5, 120.2)
- added D2: D_Schottky, Diode_THT:D_DO-201AD_P15.24mm_Horizontal, F.Cu at (116.9, 57.2)
- added R1: 10k, Resistor_THT:R_Axial_DIN0207_L6.3mm_D2.5mm_P10.16mm_Horizontal, F.Cu at (136.8, 89.7)
- added R2: 220, Resistor_THT:R_Axial_DIN0207_L6.3mm_D2.5mm_P10.16mm_Horizontal, F.Cu at (154.8, 89.8)
- added R3: 0.1R, Resistor_THT:R_Axial_Power_L25.0mm_W9.0mm_P27.94mm, F.Cu at (118.5, 82.0)
- added U1: LM7805_TO220, Package_TO_SOT_THT:TO-220-3_Vertical, F.Cu at (121.5, 114.0)
- moved J6 63.4 mm to (189.9, 56.5)
- moved J3 37.9 mm to (98.5, 113.8)
- moved J4 31.1 mm to (99.0, 57.5)
- moved Q1 14.2 mm to (129.1, 77.0)
Connections:
- J1 pad 6: /COIL_CURRENT -> /I_COIL
- J3 pad 1: /+5V -> /+12V
- Q1 pad 3: GND -> /I_COIL
Routing:
- net /+5V: track 142.4 -> 46.8 mm
- net /I_COIL: track 0.00 -> 41.6 mm
- net /HALL_OUT: track 62.6 -> 27.2 mm
- net /+12V: track 0.00 -> 28.9 mm
- net Net-(D2-A): track 25.6 -> 5.50 mm
- net /COIL_CURRENT: track 18.3 -> 0.00 mm
- net Net-(J5-Pin_2): track 13.7 -> 0.00 mm
- net /PWM_OUT: track 13.1 -> 5.33 mm
- net Net-(D2-K): track 12.9 -> 18.4 mm
- removed copper zone on B.Cu, net GND
Other:
- board text added: "+12V"
- board text removed: "+5V"
- board text removed: "CURRENT SENSOR"

Commit message: more PCB updates
Parts:
- added C4: 100nF, Capacitor_THT:C_Disc_D3.0mm_W1.6mm_P2.50mm, F.Cu at (110.8, 99.8)
- added R4: 1k, Resistor_THT:R_Axial_DIN0207_L6.3mm_D2.5mm_P10.16mm_Horizontal, F.Cu at (106.2, 89.7)
- added R5: 1k, Resistor_THT:R_Axial_DIN0207_L6.3mm_D2.5mm_P10.16mm_Horizontal, F.Cu at (132.5, 95.6)
- added R6: 15k, Resistor_THT:R_Axial_DIN0207_L6.3mm_D2.5mm_P10.16mm_Horizontal, F.Cu at (117.7, 86.0)
- added U2: MCP6002-xMC, Package_DIP:DIP-8_W7.62mm, F.Cu at (117.7, 91.7)
- moved D2 32.9 mm to (84.0, 56.4), turned to -90 degrees
- moved J3 27.7 mm to (70.8, 113.8)
- moved J4 27.3 mm to (71.8, 58.0)
- moved Q1 22.1 mm to (121.9, 56.0), turned to 0 degrees
- moved C1 20.6 mm to (91.0, 118.3)
- moved C2 20.6 mm to (116.5, 119.3)
- moved C3 20.6 mm to (128.0, 119.0)
- moved U1 20.6 mm to (100.9, 112.8)
- moved J6 12.7 mm to (177.2, 55.5)
- moved R3 12.3 mm to (106.2, 83.0)
- moved R1 9.75 mm to (146.5, 89.9)
- moved R2 7.50 mm to (162.3, 90.0)
- moved J1 6.61 mm to (166.6, 69.8)
- moved J2 6.61 mm to (192.0, 69.8)
Connections:
- D2 pad 1: Net-(D2-K) -> /+12V
- J1 pad 3: unconnected-(J1-Pin_3-Pad3) -> /I_COIL
- J1 pad 4: unconnected-(J1-Pin_4-Pad4) -> /HALL_OUT
- J1 pad 6: /I_COIL -> unconnected-(J1-Pin_6-Pad6)
- J2 pad 5: /HALL_OUT -> unconnected-(J2-Pin_5-Pad5)
- J2 pad 7: unconnected-(J2-Pin_7-Pad7) -> GND
- J4 pad 1: Net-(D2-K) -> /+12V
- Q1 pad 3: /I_COIL -> Net-(Q1-S)
- R3 pad 1: /I_COIL -> Net-(Q1-S)
Routing:
- net /+5V: track 46.8 -> 0.00 mm
- net /I_COIL: track 41.6 -> 0.00 mm
- net /+3V3: track 37.9 -> 0.00 mm
- net /+12V: track 28.9 -> 0.28 mm
- net /HALL_OUT: track 27.2 -> 0.00 mm
- net Net-(D2-K): track 18.4 -> 0.00 mm
- net Net-(Q1-G): track 14.3 -> 0.57 mm
- net Net-(D2-A): track 5.50 -> 0.00 mm
- net /PWM_OUT: track 5.33 -> 0.13 mm
Other:
- board size 112.8 x 75.8 mm -> 140.5 x 75.8 mm

Commit message: more pcb updates
Parts:
- removed C1: 100uF, Capacitor_THT:CP_Radial_D6.3mm_P2.50mm
- removed C2: 10uF, Capacitor_THT:CP_Radial_D6.3mm_P2.50mm
- removed C3: 100nF, Capacitor_THT:C_Disc_D3.0mm_W1.6mm_P2.50mm
- removed J3: Screw_Terminal_01x02, TerminalBlock:TerminalBlock_MaiXu_MX126-5.0-02P_1x02_P5.00mm
- removed U2: MCP6002-xMC, Package_DIP:DIP-8_W7.62mm
- added J5: Screw_Terminal_01x03, TerminalBlock:TerminalBlock_MaiXu_MX126-5.0-03P_1x03_P5.00mm, F.Cu at (71.8, 108.2)
- U1: value LM7805_TO220 -> MCP6002-xP; footprint Package_TO_SOT_THT:TO-220-3_Vertical -> Package_DIP:DIP-8_W7.62mm
- moved U1 26.3 mm to (117.6, 92.5)
- moved Q1 20.5 mm to (107.9, 71.0)
Connections:
- C4 pad 2: Net-(U2A-+) -> Net-(U1A-+)
- R4 pad 2: Net-(U2A-+) -> Net-(U1A-+)
- R5 pad 2: Net-(U2A--) -> Net-(U1A--)
- R6 pad 2: Net-(U2A--) -> Net-(U1A--)
- U1 pad 1: /+12V -> /I_COIL
- U1 pad 2: GND -> Net-(U1A--)
- U1 pad 3: /+5V -> Net-(U1A-+)
Routing:
- net Net-(Q1-G): track 0.57 -> 0.00 mm
Other:
- board text added: "+5V"

Commit message: more pcb updates
Parts:
- removed U1: MCP6002-xP, Package_DIP:DIP-8_W7.62mm
- added U2: LM324N, Package_DIP:DIP-14_W7.62mm, F.Cu at (118.0, 92.0)
- R6: value 15k -> 6.8k

Commit message: cooked
Parts:
- moved Q1 8.79 mm to (113.8, 64.4), turned to -90 degrees
- moved C4 8.32 mm to (106.2, 106.8), turned to 90 degrees
- moved U2 2.77 mm to (117.6, 94.7)
Connections:
- J1 pad 3: /I_COIL -> unconnected-(J1-Pin_3-Pad3)
- J1 pad 4: /HALL_OUT -> unconnected-(J1-Pin_4-Pad4)
- J1 pad 5: unconnected-(J1-Pin_5-Pad5) -> /V_HALL
- J1 pad 6: unconnected-(J1-Pin_6-Pad6) -> /V_SHUNT
- J6 pad 1: GND -> /+3V3
- J6 pad 2: /+3V3 -> GND
- J6 pad 3: /HALL_OUT -> /V_HALL
- R6 pad 1: /I_COIL -> /V_SHUNT
- U2 pad 1: /I_COIL -> /V_SHUNT
- U2 pad 2: Net-(C4-Pad2) -> Net-(R5-Pad2)
- U2 pad 3: Net-(R5-Pad2) -> Net-(C4-Pad2)
Routing:
- net /+5V: track 0.00 -> 146.9 mm
- net /V_SHUNT: track 0.00 -> 68.8 mm
- net /+12V: track 0.00 -> 65.9 mm
- net Net-(Q1-G): track 0.00 -> 56.3 mm
- net Net-(D2-A): track 0.00 -> 47.5 mm
- net Net-(R5-Pad2): track 0.00 -> 36.6 mm
- net /V_HALL: track 0.00 -> 31.0 mm
- net Net-(Q1-S): track 0.00 -> 23.3 mm
- net /+3V3: track 0.00 -> 18.7 mm
- net Net-(C4-Pad2): track 0.00 -> 15.8 mm
- net /PWM_OUT: track 0.13 -> 4.45 mm
- added copper zone on B.Cu, net GND
